Commit message: comrrt generates 2 paths

File: data/urdf/hyq/hyq_trunk_large.urdf (robot description, URDF)
Before this commit: robot hyq_trunk_large, 1 links, 0 joints
Links:
- link base_link: geometry collision mesh filename=package://hpp-rbprm-corba/meshes/hyq/hyq_trunk.stl scale=1 1 1; visual mesh filename=package://hpp-rbprm-corba/meshes/hyq/hyq_all.stl
